File: keyboard.sch (KiCad schematic (older format))
At the start: 67 parts, among them IC1 ATMEGA32U4, J1 MINI, J2 MICRO, P1 CONN_1, P10 CONN_1, P11 CONN_1, P12 CONN_1, P13 CONN_1, P14 CONN_1, P15 CONN_1, P16 CONN_1, P17 CONN_1, P18 CONN_1, P19 CONN_1, P2 CONN_1, P20 CONN_1, P21 CONN_1, P22 CONN_1, P23 CONN_1, P24 CONN_1, P25 CONN_1, P26 CONN_1, P27 CONN_1, P28 CONN_1, P29 CONN_1, P3 CONN_1, P30 CONN_1, P31 CONN_1, P32 CONN_1, P33 CONN_1, P34 CONN_1, P35 CONN_1, P36 CONN_1, P37 CONN_1, P38 CONN_1, P39 CONN_1, P4 CONN_1, P40 CONN_1, P41 CONN_1, P42 CONN_1, P5 CONN_1, P6 CONN_1, P7 CONN_1, P8 CONN_1, P9 CONN_1, Q1 MOSFET_P, X1 CRYSTAL

Commit message: 完成
Parts:
- removed C1, C2: 22p, symbol C
- removed C3, C8: 1u, symbol C
- removed C4, C5, C6, C7: 100n, symbol C
- removed IC1: ATMEGA32U4, symbol ATMEGA32U4
- removed J1: MINI, symbol USBMINI_B05
- removed J2: MICRO, Connect:USB_Micro-B, symbol USBMINI_B05
- removed JP1, JP2, JP3, JP4, JP5, JP6: JUMPER, Resistors_SMD:R_0201, symbol JUMPER
- removed P1, P10, P11, P12, P13, P14, P15, P16, P17, P18, P19, P2, P20, P21, P22, P23, P24, P25, P26, P27, P28, P29, P3, P30, P31, P32, P33, P34, P35, P36, P37, P38, P39, P4, P40, P41, P42, P5, P6, P7, P8, P9: CONN_1, symbol CONN_1
- removed Q1: MOSFET_P, TO_SOT_Packages_SMD:SOT-23, symbol PNP
- removed R1, R2: 22, symbol R
- removed R3, R5: 10k, symbol R
- removed R65: 10k, Resistors_SMD:R_0805, symbol R
- removed S0: DTSM-6, symbol DTSM-6
- removed X1: CRYSTAL, Crystals:Crystal_HC49-U_Vertical, symbol CRYSTAL
- added C1: 22nF, Capacitor_SMD:C_0805_2012Metric, symbol keyboard-rescue:C_Small-RESCUE-ble4100-nrf-ble4100-nrf-rescue
- added C2, C3, C4: 1uF, Capacitor_SMD:C_0805_2012Metric, symbol keyboard-rescue:C_Small-RESCUE-ble4100-nrf-ble4100-nrf-rescue
- added C5: 22uF, Capacitor_SMD:C_0805_2012Metric, symbol keyboard-rescue:C_Small-RESCUE-ble4100-nrf-ble4100-nrf-rescue
- added C6, C7: 0.1uF, Capacitor_SMD:C_0805_2012Metric, symbol keyboard-rescue:C_Small-RESCUE-ble4100-nrf-ble4100-nrf-rescue
- added C8: 47pF, Capacitor_SMD:C_0805_2012Metric, symbol keyboard-rescue:C_Small-RESCUE-ble4100-nrf-ble4100-nrf-rescue
- added D20, D25, D35, D40, D45: LED, MX1A:MX1A-led, symbol device:LED
- added J1: USB_OTG, custom:USB_Micro-B_lowp, symbol conn:USB_OTG
- added K1: Jumper_NO_Small, Resistor_SMD:R_0805_2012Metric, symbol keyboard-rescue:Jumper_NO_Small-RESCUE-ble4100-nrf-ble4100-nrf-rescue
- added P2: BATT, Connector_PinHeader_2.54mm:PinHeader_1x02_P2.54mm_Vertical, symbol keyboard-rescue:CONN_01X02-RESCUE-ble4100-nrf-ble4100-nrf-rescue
- added P3: SWD, Connector_PinSocket_2.54mm:PinSocket_1x04_P2.54mm_Vertical, symbol keyboard-rescue:CONN_01X04-RESCUE-ble4100-nrf-ble4100-nrf-rescue
- added R1: 1.5K, Resistor_SMD:R_0805_2012Metric, symbol keyboard-rescue:R_Small-RESCUE-ble4100-nrf-ble4100-nrf-rescue
- added R10: 20K, Resistor_SMD:R_0805_2012Metric, symbol keyboard-rescue:R_Small-RESCUE-ble4100-nrf-ble4100-nrf-rescue
- added R2, R3, R5, R7, R9: R, Resistor_SMD:R_0805_2012Metric, symbol device:R
- added R6: 10M, Resistor_SMD:R_0805_2012Metric, symbol keyboard-rescue:R_Small-RESCUE-ble4100-nrf-ble4100-nrf-rescue
- added R8: 2.2M, Resistor_SMD:R_0805_2012Metric, symbol keyboard-rescue:R_Small-RESCUE-ble4100-nrf-ble4100-nrf-rescue
- added U1: nrf51822-02, custom:nRF51822-02, symbol keyboard-rescue:nrf51822-02-RESCUE-ble4100-nrf-ble4100-nrf-rescue
- added U2: TP4057, Package_TO_SOT_SMD:SOT-23-6, symbol keyboard-rescue:TP4057-RESCUE-ble4100-nrf-ble4100-nrf-rescue
- added U3: RT9193, Package_TO_SOT_SMD:SOT-23-5, symbol keyboard-rescue:RT9193-RESCUE-ble4100-nrf-ble4100-nrf-rescue
- added U4: CH554T, Package_SO:SSOP-20_4.4x6.5mm_P0.65mm, symbol keyboard-rescue:CH554T-ch554t
Connections:
- net labels added: 3V3, ADC1, BATT, CHRG, DCLK, DIO, RXD, STBY, TXD, UD_N, UD_P, V33, caps_led, led1, led2, led3, led4, led5
- net labels removed: GPIO0, GPIO1, GPIO2, GPIO3, MISO, MOSI, SCK, caps, ~RES~
- wire segments 178 -> 109
- no-connect marks 6 -> 16
Other:
- note added: "Key to start download, place near to UDP line."
- note added: "Power"
- note removed: "Backlight expansion\nconnector (top)"
- note removed: "Universal expansion\nconnector (bottom)"

Commit message: 细节修正
Parts:
- renumbered C6 to C1, C7 to C2, C8 to C3, C2 to C4, C3 to C5, C4 to C6, C5 to C7, C1 to C8, D20 to LED1, D25 to LED2, D35 to LED3, D40 to LED4, D45 to LED5, P3 to P1, R10 to R1, R1 to R2, R6 to R3, R8 to R4, R2 to RL1, R3 to RL2, R5 to RL3, R7 to RL4, R9 to RL5, U4 to U2, U2 to U3, U3 to U4

Commit message: 元件丢正面
Parts:
- C1, C2, C4, C5, C6: symbol keyboard-rescue:C_Small-RESCUE-ble4100-nrf-ble4100-nrf-rescue -> Device:C_Small
- C3: value 47pF -> NC/47pF; symbol keyboard-rescue:C_Small-RESCUE-ble4100-nrf-ble4100-nrf-rescue -> Device:C_Small
- C7: value 22uF -> 10nF; symbol keyboard-rescue:C_Small-RESCUE-ble4100-nrf-ble4100-nrf-rescue -> Device:C_Small
- J1: symbol conn:USB_OTG -> Connector_Specialized:USB_B_Mini
- LED1, LED2, LED3, LED4, LED5: symbol device:LED -> Device:LED
- RL1, RL2, RL3, RL4, RL5: symbol device:R -> Device:R
Changed lines of the file:
@@
 $EndComp
 $Comp
-L keyboard-rescue:C_Small-RESCUE-ble4100-nrf-ble4100-nrf-rescue C5
+L Device:C_Small C5
 U 1 1 58689C6E
 P 7900 5750
@@
 $EndComp
 $Comp
-L keyboard-rescue:C_Small-RESCUE-ble4100-nrf-ble4100-nrf-rescue C6
+L Device:C_Small C6
 U 1 1 58689C99
 P 8100 5750
@@
 $EndComp
 $Comp
-L keyboard-rescue:C_Small-RESCUE-ble4100-nrf-ble4100-nrf-rescue C4
+L Device:C_Small C4
 U 1 1 5868B8D5
 P 7650 5750
@@
 $EndComp
 $Comp
-L keyboard-rescue:C_Small-RESCUE-ble4100-nrf-ble4100-nrf-rescue C7
+L Device:C_Small C7
 U 1 1 5869898F
 P 8700 5750
 F 0 "C7" H 8710 5820 50  0000 L CNN
-F 1 "22uF" H 8710 5670 50  0000 L CNN
+F 1 "10nF" H 8710 5670 50  0000 L CNN
 F 2 "Capacitor_SMD:C_0805_2012Metric" H 8700 5750 50  0001 C CNN
 F 3 "" H 8700 5750 50  0000 C CNN
@@
 $EndComp
 $Comp
-L keyboard-rescue:C_Small-RESCUE-ble4100-nrf-ble4100-nrf-rescue C1
+L Device:C_Small C1
 U 1 1 5A0D902C
 P 1550 6000
@@
 $EndComp
 $Comp
-L keyboard-rescue:C_Small-RESCUE-ble4100-nrf-ble4100-nrf-rescue C2
+L Device:C_Small C2
 U 1 1 5A0D91A2
 P 1850 6000
@@
 $EndComp
 $Comp
-L keyboard-rescue:C_Small-RESCUE-ble4100-nrf-ble4100-nrf-rescue C3
+L Device:C_Small C3
 U 1 1 5A0DBAA2
 P 3100 6350
 F 0 "C3" H 3110 6420 50  0000 L CNN
-F 1 "47pF" H 3110 6270 50  0000 L CNN
+F 1 "NC/47pF" H 3110 6270 50  0000 L CNN
 F 2 "Capacitor_SMD:C_0805_2012Metric" H 3100 6350 50  0001 C CNN
 F 3 "" H 3100 6350 50  0000 C CNN
@@
 	1    0    0    -1
 $EndComp
-Text GLabel 3700 6200 2    60   Input ~ 0
-VCC
 Text GLabel 2700 6200 0    60   Input ~ 0
 UD_P
@@
 	1    0    0    -1
 $EndComp
-Text GLabel 2300 3200 3    60   Input ~ 0
+Text GLabel 3000 3200 3    60   Input ~ 0
 RXD
-Text GLabel 2400 3200 3    60   Input ~ 0
+Text GLabel 3550 2850 2    60   Input ~ 0
 TXD
 Wire Bus Line
@@
 	2800 3400 2900 3500
 Entry Wire Line
-	2900 3400 3000 3500
-Entry Wire Line
-	3000 3400 3100 3500
+	2500 3400 2600 3500
 Entry Wire Line
 	3850 1650 3950 1750
@@
 	3850 2550 3950 2650
 Entry Wire Line
-	3850 2850 3950 2950
+	2400 3400 2500 3500
 Wire Wire Line
 	3550 1650 3850 1650
@@
 Wire Wire Line
 	3850 2550 3550 2550
-Wire Wire Line
-	3550 2850 3850 2850
-Wire Wire Line
-	3000 3200 3000 3400
-Wire Wire Line
-	2900 3400 2900 3200
 Wire Wire Line
 	2800 3200 2800 3400
@@
 Wire Wire Line
 	3000 1100 3000 1300
+Text Label 2800 3350 1    50   ~ 0
+row1
+Text Label 2700 3350 1    50   ~ 0
+row2
+Text Label 2600 3350 1    50   ~ 0
+row3
+Text Label 2500 3350 1    50   ~ 0
+row4
+Text Label 2400 3350 1    50   ~ 0
+row5
+Text Label 3550 2650 0    50   ~ 0
+col1
+Text Label 3550 2450 0    50   ~ 0
+col2
+Text Label 3550 2250 0    50   ~ 0
+col3
+Text Label 3550 2050 0    50   ~ 0
+col4
+Text Label 3550 1850 0    50   ~ 0
+col5
+Text Label 3550 1650 0    50   ~ 0
+col6
+Text Label 2900 1300 1    50   ~ 0
+col7
+Text Label 2800 1300 1    50   ~ 0
+col8
+Text Label 2700 1300 1    50   ~ 0
+col9
 Text Label 2600 1300 1    50   ~ 0
-row1
+col10
 Text Label 2500 1300 1    50   ~ 0
-row2
+col11
 Text Label 2400 1300 1    50   ~ 0
-row3
+col12
 Text Label 2300 1300 1    50   ~ 0
-row4
+col13
 Text Label 2200 1300 1    50   ~ 0
-row5
-Text Label 2700 1300 1    50   ~ 0
-col1
-Text Label 2800 1300 1    50   ~ 0
-col2
-Text Label 2900 1300 1    50   ~ 0
-col3
+col14
+Text Label 3550 2550 0    50   ~ 0
+caps_led
+Text Label 3550 2350 0    50   ~ 0
+led1
+Text Label 3550 2150 0    50   ~ 0
+led2
+Text Label 3550 1950 0    50   ~ 0
+led3
+Text Label 3550 1750 0    50   ~ 0
+led4
 Text Label 3000 1300 1    50   ~ 0
-col4
-Text Label 3550 1650 0    50   ~ 0
-col5
-Text Label 3550 1750 0    50   ~ 0
-col6
-Text Label 3550 1850 0    50   ~ 0
-col7
-Text Label 3550 1950 0    50   ~ 0
-col8
-Text Label 3550 2050 0    50   ~ 0
-col9
-Text Label 3550 2150 0    50   ~ 0
-col10
-Text Label 3550 2250 0    50   ~ 0
-col11
-Text Label 3550 2350 0    50   ~ 0
-col12
-Text Label 3550 2450 0    50   ~ 0
-col13
-Text Label 3550 2550 0    50   ~ 0
-col14
-Text Label 2600 3400 1    50   ~ 0
-caps_led
-Text Label 2700 3400 1    50   ~ 0
-led1
-Text Label 2800 3400 1    50   ~ 0
-led2
-Text Label 2900 3400 1    50   ~ 0
-led3
-Text Label 3000 3400 1    50   ~ 0
-led4
-Text Label 3750 2850 2    50   ~ 0
 led5
 Entry Wire Line
@@
 	5400 3850 5150 3850
 $Comp
-L device:LED LED1
+L Device:LED LED1
 U 1 1 5A98E30A
 P 6000 4450
@@
 $EndComp
 $Comp
-L device:R RL1
+L Device:R RL1
 U 1 1 5A98E673
 P 5600 4450
@@
 	5750 4450 5850 4450
 $Comp
-L device:LED LED2
+L Device:LED LED2
 U 1 1 5A9996E8
 P 6000 4800
@@
 $EndComp
 $Comp
-L device:R RL2
+L Device:R RL2
 U 1 1 5A9996EF
 P 5600 4800
@@
 	5750 4800 5850 4800
 $Comp
-L device:LED LED3
+L Device:LED LED3
 U 1 1 5A99C333
 P 6000 5150
@@
 $EndComp
 $Comp
-L device:R RL3
+L Device:R RL3
 U 1 1 5A99C33A
 P 5600 5150
@@
 	5750 5150 5850 5150
 $Comp
-L device:LED LED4
+L Device:LED LED4
 U 1 1 5A99F1F4
 P 6000 5500
@@
 $EndComp
 $Comp
-L device:R RL4
+L Device:R RL4
 U 1 1 5A99F1FB
 P 5600 5500
@@
 	5750 5500 5850 5500
 $Comp
-L device:LED LED5
+L Device:LED LED5
 U 1 1 5A9A1FE2
 P 6000 5850
@@
 $EndComp
 $Comp
-L device:R RL5
+L Device:R RL5
 U 1 1 5A9A1FE9
 P 5600 5850
@@
 	6300 5850 6300 6150
 NoConn ~ 3550 2750
-NoConn ~ 3550 2650
-NoConn ~ 2500 3200
-$Comp
-L conn:USB_OTG J1
+$Comp
+L Connector_Specialized:USB_B_Mini J1
 U 1 1 5AA225CF
 P 1350 5250
@@
 Text GLabel 2200 3200 3    60   Input ~ 0
 ADC1
+Text GLabel 3700 6200 2    60   Input ~ 0
+V33
+Wire Wire Line
+	2500 3200 2500 3400
+Wire Wire Line
+	2400 3400 2400 3200
+NoConn ~ 2300 3200
+Entry Wire Line
+	3850 2650 3950 2750
+Wire Wire Line
+	3550 2650 3850 2650
+NoConn ~ 2900 3200
 Wire Bus Line
 	1200 3500 3950 3500

Commit message: 修改
Parts:
- removed C8: 22nF, Capacitor_SMD:C_0805_2012Metric, symbol keyboard-rescue:C_Small-RESCUE-ble4100-nrf-ble4100-nrf-rescue
- removed U4: RT9193, Package_TO_SOT_SMD:SOT-23-5, symbol keyboard-rescue:RT9193-RESCUE-ble4100-nrf-ble4100-nrf-rescue
- added U4: XC6206P30, Package_TO_SOT_SMD:SOT-23, symbol Regulator_Linear:AP2127N-3.0
Connections:
- wire segments 109 -> 104
Changed lines of the file:
@@
-$EndComp
-$Comp
-L keyboard-rescue:RT9193-RESCUE-ble4100-nrf-ble4100-nrf-rescue U4
-U 1 1 58687662
-P 10250 4850
-F 0 "U4" H 10250 4650 60  0000 C CNN
-F 1 "RT9193" H 10250 4750 60  0000 C CNN
-F 2 "Package_TO_SOT_SMD:SOT-23-5" H 10200 4850 60  0001 C CNN
-F 3 "" H 10200 4850 60  0001 C CNN
-	1    10250 4850
-	1    0    0    -1
 $EndComp
 $Comp
@@
 Text GLabel 8800 4300 2    60   Input ~ 0
 BATT
-Text GLabel 9800 4600 0    60   Input ~ 0
-BATT
 Text GLabel 10500 3700 0    60   Input ~ 0
 BATT
-$Comp
-L keyboard-rescue:GND-RESCUE-ble4100-nrf-ble4100-nrf-rescue #PWR016
-U 1 1 5868900A
-P 9550 5150
-F 0 "#PWR016" H 9550 4900 50  0001 C CNN
-F 1 "GND" H 9550 5000 50  0000 C CNN
-F 2 "" H 9550 5150 50  0000 C CNN
-F 3 "" H 9550 5150 50  0000 C CNN
-	1    9550 5150
-	1    0    0    -1
-$EndComp
-Text GLabel 10700 4600 2    60   Input ~ 0
-3V3
 Text GLabel 1750 4500 2    60   Input ~ 0
 3V3
@@
 DCLK
 $Comp
-L keyboard-rescue:C_Small-RESCUE-ble4100-nrf-ble4100-nrf-rescue C8
-U 1 1 58689C31
-P 10750 4950
-F 0 "C8" H 10760 5020 50  0000 L CNN
-F 1 "22nF" H 10760 4870 50  0000 L CNN
-F 2 "Capacitor_SMD:C_0805_2012Metric" H 10750 4950 50  0001 C CNN
-F 3 "" H 10750 4950 50  0000 C CNN
-	1    10750 4950
-	1    0    0    -1
-$EndComp
-$Comp
 L Device:C_Small C5
 U 1 1 58689C6E
@@
 F 3 "" H 8100 5750 50  0000 C CNN
 	1    8100 5750
-	1    0    0    -1
-$EndComp
-$Comp
-L keyboard-rescue:GND-RESCUE-ble4100-nrf-ble4100-nrf-rescue #PWR018
-U 1 1 5868A007
-P 10750 5150
-F 0 "#PWR018" H 10750 4900 50  0001 C CNN
-F 1 "GND" H 10750 5000 50  0000 C CNN
-F 2 "" H 10750 5150 50  0000 C CNN
-F 3 "" H 10750 5150 50  0000 C CNN
-	1    10750 5150
 	1    0    0    -1
 $EndComp
@@
 	10450 3800 10450 4000
 Wire Wire Line
-	9800 4700 9550 4700
-Wire Wire Line
 	1750 4200 1850 4200
 Wire Wire Line
@@
 Connection ~ 1550 2850
 Wire Wire Line
-	10700 4800 10750 4800
-Wire Wire Line
 	7850 4400 7900 4400
 Wire Wire Line
 	7650 5850 7650 5950
-Wire Wire Line
-	9550 4700 9550 5150
 Wire Wire Line
 	7650 4400 7550 4400
@@
 	8950 5350 8950 5300
 Connection ~ 8700 5600
-Wire Wire Line
-	10750 4800 10750 4850
-Wire Wire Line
-	10750 5050 10750 5150
 Wire Notes Line
 	7300 2700 11200 2700
@@
 	8000 5900 8000 5950
 Connection ~ 8000 5900
-Text GLabel 9800 4800 0    60   Input ~ 0
-BATT
 $Comp
 L keyboard-rescue:CH554T-ch554t U2
@@
 	3550 2650 3850 2650
 NoConn ~ 2900 3200
+$Comp
+L Regulator_Linear:AP2127N-3.0 U4
+U 1 1 5AE6D677
+P 10250 4750
+F 0 "U4" H 10250 4992 50  0000 C CNN
+F 1 "XC6206P30" H 10250 4901 50  0000 C CNN
+F 2 "Package_TO_SOT_SMD:SOT-23" H 10250 4975 50  0001 C CIN
+F 3 "https://www.diodes.com/assets/Datasheets/AP2127.pdf" H 10250 4750 50  0001 C CNN
+	1    10250 4750
+	1    0    0    -1
+$EndComp
+Text GLabel 9950 4750 0    60   Input ~ 0
+BATT
+Text GLabel 10550 4750 2    60   Input ~ 0
+3V3
+$Comp
+L keyboard-rescue:GND-RESCUE-ble4100-nrf-ble4100-nrf-rescue #PWR016
+U 1 1 5AE6D8BF
+P 10250 5050
+F 0 "#PWR016" H 10250 4800 50  0001 C CNN
+F 1 "GND" H 10250 4900 50  0000 C CNN
+F 2 "" H 10250 5050 50  0000 C CNN
+F 3 "" H 10250 5050 50  0000 C CNN
+	1    10250 5050
+	1    0    0    -1
+$EndComp
 Wire Bus Line
 	1200 3500 3950 3500

Commit message: 修正几个问题
修正ADC接口不正确的问题
增加防反冲二极管
Parts:
- added D20: SS14, Diode_SMD:D_0805_2012Metric, symbol Device:D
- R1: value 20K -> 10K
- R2: value 1.5K -> 4.7K
Connections:
- wire segments 104 -> 105
Changed lines of the file:
@@
 P 7750 4400
 F 0 "R2" H 7780 4420 50  0000 L CNN
-F 1 "1.5K" H 7780 4360 50  0000 L CNN
+F 1 "4.7K" H 7780 4360 50  0000 L CNN
 F 2 "Resistor_SMD:R_0805_2012Metric" H 7750 4400 50  0001 C CNN
 F 3 "" H 7750 4400 50  0000 C CNN
@@
 Text Notes 9150 6450 0    60   ~ 0
 Power
-Text GLabel 8800 4200 2    60   Input ~ 0
+Text GLabel 9100 4200 2    60   Input ~ 0
 VCC
 Text GLabel 7650 5650 1    60   Input ~ 0
@@
 P 2950 6200
 F 0 "R1" H 2980 6220 50  0000 L CNN
-F 1 "20K" H 2980 6160 50  0000 L CNN
+F 1 "10K" H 2980 6160 50  0000 L CNN
 F 2 "Resistor_SMD:R_0805_2012Metric" H 2950 6200 50  0001 C CNN
 F 3 "" H 2950 6200 50  0000 C CNN
@@
 	1200 1000 1200 3500
 Entry Wire Line
-	2100 1000 2200 1100
-Entry Wire Line
-	2200 1000 2300 1100
+	2200 3400 2300 3500
 Entry Wire Line
 	2300 1000 2400 1100
@@
 Entry Wire Line
 	2900 1000 3000 1100
-Wire Wire Line
-	2200 1300 2200 1100
 Wire Wire Line
 	2300 1100 2300 1300
@@
 Text Label 2400 1300 1    50   ~ 0
 col12
-Text Label 2300 1300 1    50   ~ 0
+Text Label 2200 1300 1    50   ~ 0
 col13
-Text Label 2200 1300 1    50   ~ 0
+Text Label 2200 3350 1    50   ~ 0
 col14
 Text Label 3550 2550 0    50   ~ 0
@@
 $EndComp
 NoConn ~ 1650 5450
-Text GLabel 2200 3200 3    60   Input ~ 0
+Text GLabel 2300 1100 1    60   Input ~ 0
 ADC1
 Text GLabel 3700 6200 2    60   Input ~ 0
@@
 	1    0    0    -1
 $EndComp
+Wire Wire Line
+	2200 3200 2200 3400
+Wire Wire Line
+	2200 1100 2200 1300
+Entry Wire Line
+	2100 1000 2200 1100
 Wire Bus Line
 	1200 3500 3950 3500
@@
 Wire Bus Line
 	5050 1300 5050 5850
+$Comp
+L Device:D D20
+U 1 1 5AFFEAFC
+P 8950 4200
+F 0 "D20" H 8950 4416 50  0000 C CNN
+F 1 "SS14" H 8950 4325 50  0000 C CNN
+F 2 "Diode_SMD:D_0805_2012Metric" H 8950 4200 50  0001 C CNN
+F 3 "~" H 8950 4200 50  0001 C CNN
+	1    8950 4200
+	1    0    0    -1
+$EndComp
 $EndSCHEMATC

Commit message: 替换接口为Type-C
Parts:
- removed J1: USB_OTG, custom:USB_Micro-B_lowp, symbol Connector_Specialized:USB_B_Mini
- added J1: USB_C_Receptacle_USB2.0, Connector_USB:USB_C_Receptacle_Amphenol_12401610E4-2A, symbol Connector:USB_C_Receptacle_USB2.0
- added R5, R6: 5.1K, Resistor_SMD:R_0805_2012Metric, symbol keyboard-rescue:R_Small-RESCUE-ble4100-nrf-ble4100-nrf-rescue
- added TP1, TP2, TP3: TP, TestPoint:TestPoint_Pad_D1.0mm, symbol Connector:TestPoint
Connections:
- net labels added: CLK, MISO, MOSI
- net labels removed: RXD, TXD
- wire segments 105 -> 109
- no-connect marks 16 -> 15
Other:
- moved on the sheet: C1, C2, C3, K1, P1, R1, U2

Commit message: 使用52810替换51822
Parts:
- removed LED4, LED5: LED, MX1A:MX1A-led, symbol Device:LED
- removed RL1, RL2, RL3, RL4, RL5: R, Resistor_SMD:R_0805_2012Metric, symbol Device:R
- removed U1: nrf51822-02, custom:nRF51822-02, symbol keyboard-rescue:nrf51822-02-RESCUE-ble4100-nrf-ble4100-nrf-rescue
- added C8: 10uF, Capacitor_SMD:C_0805_2012Metric, symbol Device:C_Small
- added J2, J3: -, Connector_PinSocket_2.54mm:PinSocket_1x05_P2.54mm_Vertical, symbol Connector:Conn_01x05_Female
- added JP1: Jumper, Jumper:SolderJumper-2_P1.3mm_Bridged2Bar_Pad1.0x1.5mm, symbol Jumper:SolderJumper_2_Bridged
- added RL1, RL2, RL3: 4.7K, Resistor_SMD:R_0805_2012Metric, symbol keyboard-rescue:R_Small-RESCUE-ble4100-nrf-ble4100-nrf-rescue
- added TP4, TP5: TP, TestPoint:TestPoint_Pad_D1.0mm, symbol Connector:TestPoint
- added U1: nRF52810-ND04C, Customv2:nRF52810-ND04C, symbol custom:nRF52810-ND04C
- C4: value 1uF -> 0.1uF
- J1: symbol Connector:USB_C_Receptacle_USB2.0 -> keyboard-rescue:USB_C_Receptacle_USB2.0-Connector
- LED1, LED2, LED3: symbol Device:LED -> Device:LED_Small
Connections:
- net 3V3: now also J3.1 (Pin_1), U1.2 (VCC)
- net ADC1: now also U1.13 (P02/AIN0)
- net CHRG: now also U2.11 (P3.3); no longer U2.2 (P1.4)
- net CLK: now also U2.5 (P1.7), U1.30 (P17); no longer U2.7 (P1.0)
- net DCLK: now also U1.29 (SWDCLK)
- net DIO: now also U1.28 (SWDIO)
- net GND: now also C8.2, J3.5 (Pin_5), U1.1 (GND)
- net MISO: now also U2.4 (P1.6), U1.31 (P18); no longer U2.5 (P1.7)
- net MOSI: now also U2.3 (P1.5), JP1.1 (A); no longer U2.4 (P1.6)
- net STBY: now also U2.12 (P3.4); no longer U2.3 (P1.5)
- net VCC: now also C8.1
- net col1: now also U1.27 (P16)
- net col10: now also U1.16 (P05/AIN3)
- net col11: now also U1.17 (P06)
- net col12: now also U1.18 (P07)
- net col13: now also U1.19 (P08)
- net col14: now also U1.20 (P09)
- net col2: now also U1.26 (P15)
- net col3: now also U1.25 (P14)
- net col4: now also U1.24 (P13)
- net col5: now also U1.23 (P12)
- net col6: now also U1.22 (P11)
- net col7: now also U1.12 (P27)
- net col8: now also U1.14 (P03/AIN1)
- net col9: now also U1.15 (P04/AIN2)
- net led1: now also RL1.2, U1.4 (P22)
- net led2: now also RL2.2, U1.5 (P23)
- net led3: now also RL3.2, U1.6 (P24)
- net row1: now also J2.1 (Pin_1), U1.7 (P25)
- net row2: now also J2.2 (Pin_2), U1.8 (P28/AIN4)
- net row3: now also J2.3 (Pin_3), U1.9 (P29/AIN5)
- net row4: now also J2.4 (Pin_4), U1.10 (P30/AIN6)
- net row5: now also J2.5 (Pin_5), U1.11 (P26)
- net D_RX: now reaches U2.10 (P3.0)
- net D_RX: now also TP4.1
- net D_TX: now reaches U2.9 (P3.1)
- net D_TX: now also TP5.1
- net at LED1.2 (A): now also RL1.1
- net at LED2.2 (A): now also RL2.1
- net at LED3.2 (A): now also RL3.1
- new net GPIO0: J3.2 (Pin_2), U1.21 (P10)
- new net GPIO1: J3.3 (Pin_3), U1.33 (P20)
- new net GPIO2: J3.4 (Pin_4), JP1.2 (B), U1.32 (P19)
- new net caps: U1.3 (P21/RESET)
- no-connect marks 15 -> 10
Other:
- moved on the sheet: LED1, LED2, LED3, TP1, TP2, TP3

Commit message: 微调布线
Other:
- note added: "I_{chrg} = 1000/R2"
Changed lines of the file:
@@
 Text GLabel 5400 6450 0    60   Input ~ 0
 3V3
+Text Notes 7750 4850 0    50   ~ 0
+I_{chrg} = 1000/R2
 Wire Bus Line
 	2100 1250 3850 1250
